Commit message: modify wrist link

File: arm_description/urdf/arm.xacro (robot description, xacro)
@@ -10,5 +10,6 @@
   <xacro:property name="l_link_length_2" value=".22" /> <!-- Link 1 -->
   <xacro:property name="r_link_length_2" value=".18" /> <!-- Link 1 -->
-  <xacro:property name="r_link_length_4" value=".22" /> <!-- Link 1 -->
+  <xacro:property name="r_link_length_3" value=".22" /> <!-- Link 1 -->
+  <xacro:property name="r_link_length_4" value=".02" /> <!-- Link 1 -->
   <xacro:property name="body_height" value="0.7" />  <!-- 1.3 -0.4 -->
   <xacro:property name="height1" value="2" /> <!-- Link 1 -->
@@ -92,14 +93,8 @@
   </joint>
   <link name="r_s_link_3">
-    <collision>
-      <origin xyz="0 0 0" rpy="0 0 0"/>
+    <visual>
+      <origin xyz="0 0 ${r_link_length_3/2}" rpy="0 0 0"/>
       <geometry>
-	<box size="0 0 0"/>
-      </geometry>
-    </collision>
-    <visual>
-      <origin xyz="0 0 0" rpy="0 0 0"/>
-      <geometry>
-	<box size="0 0 0"/>
+	<box size="${link_width} ${link_width} ${r_link_length_3}"/>
       </geometry>
       <material name="white"/>
@@ -113,16 +108,10 @@
   </joint>
   <link name="r_s_link_4">
-    <collision>
-      <origin xyz="0 0 ${r_link_length_4/2}" rpy="0 0 0"/>
+    <visual>
+      <origin xyz="0 0 ${r_link_length_3 + r_link_length_4/2}" rpy="0 0 0"/>
       <geometry>
-	<box size="${link_width} ${link_width} ${r_link_length_4}"/>
+        <box size="${link_width} ${link_width} ${r_link_length_4}"/>
       </geometry>
-    </collision>
-    <visual>
-      <origin xyz="0 0 ${r_link_length_4/2}" rpy="0 0 0"/>
-      <geometry>
-	<box size="${link_width} ${link_width} ${r_link_length_4}"/>
-      </geometry>
-      <material name="white"/>
+      <material name="yellow"/>
     </visual>
   </link>
